Commit message: Edit arm urdf

File: avatar_description/urdf/follower/follower_arm.urdf.xacro (robot description, xacro)
@@ -33,4 +33,5 @@
       </inertial>
     </link>
+    <!-- right arm -->
     <!-- joint1 -->
     <joint name="${prefix}right_joint1" type="revolute">
@@ -118,5 +119,5 @@
       </visual>
       <collision>
-        <origin xyz="${robot_thickness/2} 0 0" rpy="${pi/2} 0 0" />
+        <origin xyz="0 0 ${-robot_thickness/2}" rpy="${pi/2} 0 ${pi/2}" />
         <geometry>
           <cylinder radius="${robot_thickness/2}" length="${robot_thickness}"/>
@@ -182,5 +183,5 @@
       </visual>
       <collision>
-        <origin xyz="${robot_thickness/2} 0 0" rpy="${pi/2} 0 0" />
+        <origin xyz="0 0 ${-robot_thickness/2}" rpy="${pi/2} 0 ${pi/2}" />
         <geometry>
           <cylinder radius="${robot_thickness/2}" length="${robot_thickness}"/>
@@ -225,4 +226,262 @@
       </inertial>
     </link>
+    <!-- left arm -->
+    <!-- joint1 -->
+    <joint name="${prefix}left_joint1" type="revolute">
+      <parent link="${prefix}link0" />
+      <child link="${prefix}left_link1" />
+      <origin xyz="${-body_width/2} 0 ${body_height - robot_thickness/2}" rpy="0 0 0" />
+      <axis xyz="1 0 0" />
+      <limit velocity="4.8" effort="1000" lower="${-pi}" upper="${pi}" />
+      <dynamics damping="0.05" />
+    </joint>
+    <!-- link1 -->
+    <link name="${prefix}left_link1" >
+      <visual>
+        <origin xyz="${-robot_thickness/2} 0 0" rpy="${pi/2} 0 0" />
+        <geometry>
+          <cylinder radius="${robot_thickness/2}" length="${robot_thickness}"/>
+        </geometry>
+        <material name="grey">
+          <color rgba="0.2 0.2 0.2 1" />
+        </material>
+      </visual>
+      <collision>
+        <origin xyz="${-robot_thickness/2} 0 0" rpy="${pi/2} 0 0" />
+        <geometry>
+          <cylinder radius="${robot_thickness/2}" length="${robot_thickness}"/>
+        </geometry>
+      </collision>
+      <inertial>
+        <origin xyz="0 0 0.05" />
+        <mass value="1.0e-1" />
+        <inertia ixx="5e-5" ixy="0" ixz="0" iyy="5e-5" iyz="0" izz="1e-5" />
+      </inertial>
+    </link>
+    <!-- joint2 -->
+    <joint name="${prefix}left_joint2" type="revolute">
+      <parent link="${prefix}left_link1" />
+      <child link="${prefix}left_link2" />
+      <origin xyz="${-robot_thickness/2} 0 0" rpy="0 0 0" />
+      <axis xyz="0 1 0" />
+      <limit velocity="4.8" effort="1000" lower="${-pi/2}" upper="${-pi}" />
+      <dynamics damping="0.1" />
+    </joint>
+    <!-- link2 -->
+    <link name="${prefix}left_link2" >
+      <visual>
+        <origin xyz="0 0 ${-robot_thickness/2 - arm1_height/2}" rpy="0 0 0" />
+        <geometry>
+          <box size="${robot_thickness} ${robot_thickness} ${arm1_height}" />
+        </geometry>
+        <material name="grey">
+          <color rgba="0.2 0.2 0.2 1" />
+        </material>
+      </visual>
+      <collision>
+        <origin xyz="0 0 ${-robot_thickness/2 - arm1_height/2}" rpy="0 0 0" />
+        <geometry>
+          <box size="${robot_thickness} ${robot_thickness} ${arm1_height}" />
+        </geometry>
+      </collision>
+      <inertial>
+        <origin xyz="0 0 0.05" />
+        <mass value="8.0e-2" />
+        <inertia ixx="4e-5" ixy="0" ixz="0" iyy="4e-5" iyz="0" izz="8e-6" />
+      </inertial>
+    </link>
+    <!-- joint3 -->
+    <joint name="${prefix}left_joint3" type="revolute">
+      <parent link="${prefix}left_link2" />
+      <child link="${prefix}left_link3" />
+      <origin xyz="0 0 ${-arm1_height - robot_thickness/2}" rpy="0 0 0" />
+      <axis xyz="0 0 -1" />
+      <limit velocity="4.8" effort="1000" lower="${-pi/2}" upper="${pi/2}" />
+      <dynamics damping="0.1" />
+    </joint>
+    <!-- link3 -->
+    <link name="${prefix}left_link3" >
+      <visual>
+        <origin xyz="0 0 ${-robot_thickness/2}" rpy="${pi/2} 0 ${pi/2}" />
+        <geometry>
+          <cylinder radius="${robot_thickness/2}" length="${robot_thickness}"/>
+        </geometry>
+        <material name="grey">
+          <color rgba="0.2 0.2 0.2 1" />
+        </material>
+      </visual>
+      <collision>
+        <origin xyz="0 0 ${-robot_thickness/2}" rpy="${pi/2} 0 ${pi/2}" />
+        <geometry>
+          <cylinder radius="${robot_thickness/2}" length="${robot_thickness}"/>
+        </geometry>
+      </collision>
+      <inertial>
+        <origin xyz="0 0 0.05" />
+        <mass value="1.0e-1" />
+        <inertia ixx="5e-5" ixy="0" ixz="0" iyy="5e-5" iyz="0" izz="1e-5" />
+      </inertial>
+    </link>
+    <!-- joint4 -->
+    <joint name="${prefix}left_joint4" type="revolute">
+      <parent link="${prefix}left_link3" />
+      <child link="${prefix}left_link4" />
+      <origin xyz="0 0 ${-robot_thickness/2}" rpy="0 0 0" />
+      <axis xyz="1 0 0" />
+      <limit velocity="4.8" effort="1000" lower="0" upper="${pi}" />
+      <dynamics damping="0.1" />
+    </joint>
+    <!-- link4 -->
+    <link name="${prefix}left_link4" >
+      <visual>
+        <origin xyz="0 0 ${-robot_thickness/2 - arm2_height/2}" rpy="0 0 0" />
+        <geometry>
+          <box size="${robot_thickness} ${robot_thickness} ${arm2_height}" />
+        </geometry>
+        <material name="grey">
+          <color rgba="0.2 0.2 0.2 1" />
+        </material>
+      </visual>
+      <collision>
+        <origin xyz="0 0 ${-robot_thickness/2 - arm2_height/2}" rpy="0 0 0" />
+        <geometry>
+          <box size="${robot_thickness} ${robot_thickness} ${arm2_height}" />
+        </geometry>
+      </collision>
+      <inertial>
+        <origin xyz="0 0 0.05" />
+        <mass value="8.0e-2" />
+        <inertia ixx="4e-5" ixy="0" ixz="0" iyy="4e-5" iyz="0" izz="8e-6" />
+      </inertial>
+    </link>
+     <!-- joint5 -->
+    <joint name="${prefix}left_joint5" type="revolute">
+      <parent link="${prefix}left_link4" />
+      <child link="${prefix}left_link5" />
+      <origin xyz="0 0 ${-arm2_height - robot_thickness/2}" rpy="0 0 0" />
+      <axis xyz="0 0 -1" />
+      <limit velocity="4.8" effort="1000" lower="${-pi/2}" upper="${pi/2}" />
+      <dynamics damping="0.1" />
+    </joint>
+    <!-- link5 -->
+    <link name="${prefix}left_link5" >
+      <visual>
+        <origin xyz="0 0 ${-robot_thickness/2}" rpy="${pi/2} 0 ${pi/2}" />
+        <geometry>
+          <cylinder radius="${robot_thickness/2}" length="${robot_thickness}"/>
+        </geometry>
+        <material name="grey">
+          <color rgba="0.2 0.2 0.2 1" />
+        </material>
+      </visual>
+      <collision>
+        <origin xyz="0 0 ${-robot_thickness/2}" rpy="${pi/2} 0 ${pi/2}" />
+        <geometry>
+          <cylinder radius="${robot_thickness/2}" length="${robot_thickness}"/>
+        </geometry>
+      </collision>
+      <inertial>
+        <origin xyz="0 0 0.05" />
+        <mass value="1.0e-1" />
+        <inertia ixx="5e-5" ixy="0" ixz="0" iyy="5e-5" iyz="0" izz="1e-5" />
+      </inertial>
+    </link>
+    <!-- joint6 -->
+    <joint name="${prefix}left_joint6" type="revolute">
+      <parent link="${prefix}left_link5" />
+      <child link="${prefix}left_link6" />
+      <origin xyz="0 0 ${-robot_thickness/2}" rpy="0 0 0" />
+      <axis xyz="1 0 0" />
+      <limit velocity="4.8" effort="1000" lower="${-pi/2}" upper="${pi/2}" />
+      <dynamics damping="0.1" />
+    </joint>
+    <!-- link6 -->
+    <link name="${prefix}left_link6" >
+      <visual>
+        <origin xyz="0 0 ${-robot_thickness/2 - gripper_height/2}" rpy="0 0 0" />
+        <geometry>
+          <box size="${robot_thickness} ${robot_thickness} ${gripper_height}" />
+        </geometry>
+        <material name="grey">
+          <color rgba="0.2 0.2 0.2 1" />
+        </material>
+      </visual>
+      <collision>
+        <origin xyz="0 0 ${-robot_thickness/2 - gripper_height/2}" rpy="0 0 0" />
+        <geometry>
+          <box size="${robot_thickness} ${robot_thickness} ${gripper_height}" />
+        </geometry>
+      </collision>
+      <inertial>
+        <origin xyz="0 0 0.05" />
+        <mass value="8.0e-2" />
+        <inertia ixx="4e-5" ixy="0" ixz="0" iyy="4e-5" iyz="0" izz="8e-6" />
+      </inertial>
+    </link>
+    <!-- neck -->
+    <!-- joint1 -->
+    <joint name="${prefix}neck_joint1" type="revolute">
+      <parent link="${prefix}link0" />
+      <child link="${prefix}neck_link1" />
+      <origin xyz="0 0 ${body_height}" rpy="0 0 0" />
+      <axis xyz="1 0 0" />
+      <limit velocity="4.8" effort="1000" lower="${-pi/2}" upper="${pi/2}" />
+      <dynamics damping="0.1" />
+    </joint>
+    <!-- link1 -->
+    <link name="${prefix}neck_link1" >
+      <visual>
+        <origin xyz="0 0 ${robot_thickness/2}" rpy="0 0 0" />
+        <geometry>
+          <cylinder radius="${robot_thickness/2}" length="${robot_thickness}"/>
+        </geometry>
+        <material name="grey">
+          <color rgba="0.2 0.2 0.2 1" />
+        </material>
+      </visual>
+      <collision>
+        <origin xyz="0 0 ${robot_thickness/2}" rpy="0 0 0" />
+        <geometry>
+          <cylinder radius="${robot_thickness/2}" length="${robot_thickness}"/>
+        </geometry>
+      </collision>
+      <inertial>
+        <origin xyz="0 0 0.05" />
+        <mass value="1.0e-1" />
+        <inertia ixx="5e-5" ixy="0" ixz="0" iyy="5e-5" iyz="0" izz="1e-5" />
+      </inertial>
+    </link>
+    <!-- joint2 -->
+    <joint name="${prefix}neck_joint2" type="revolute">
+      <parent link="${prefix}neck_link1" />
+      <child link="${prefix}neck_link2" />
+      <origin xyz="0 0 ${robot_thickness}" rpy="0 0 0" />
+      <axis xyz="0 0 1" />
+      <limit velocity="4.8" effort="1000" lower="${-pi/2}" upper="${pi/2}" />
+      <dynamics damping="0.1" />
+    </joint>
+    <!-- link2 -->
+    <link name="${prefix}neck_link2" >
+      <visual>
+        <origin xyz="0 0 ${robot_thickness/2}" rpy="${pi/2} 0 ${pi/2}" />
+        <geometry>
+          <cylinder radius="${robot_thickness/2}" length="${robot_thickness}"/>
+        </geometry>
+        <material name="grey">
+          <color rgba="0.2 0.2 0.2 1" />
+        </material>
+      </visual>
+      <collision>
+        <origin xyz="0 0 ${-robot_thickness/2}" rpy="${pi/2} 0 ${pi/2}" />
+        <geometry>
+          <cylinder radius="${robot_thickness/2}" length="${robot_thickness}"/>
+        </geometry>
+      </collision>
+      <inertial>
+        <origin xyz="0 0 0.05" />
+        <mass value="1.0e-1" />
+        <inertia ixx="5e-5" ixy="0" ixz="0" iyy="5e-5" iyz="0" izz="1e-5" />
+      </inertial>
+    </link>
   </xacro:macro>
 </robot>
