Commit message: Edit gazebo, ros2control

File: avatar_description/gazebo/follower.gazebo.xacro (robot description, xacro)
@@ -25,8 +25,24 @@
     </xacro:macro>
     <xacro:Link reference="${prefix}link0"/>
-    <xacro:Link reference="${prefix}link1"/>
-    <xacro:Link reference="${prefix}link2"/>
-    <xacro:SimpleTransmission trans="${prefix}trans1" joint="${prefix}joint1" actuator="${prefix}actuator1" />
-    <xacro:SimpleTransmission trans="${prefix}trans2" joint="${prefix}joint2" actuator="${prefix}actuator2" />
+    <xacro:Link reference="${prefix}right_link1"/>
+    <xacro:Link reference="${prefix}right_link2"/>
+    <xacro:Link reference="${prefix}right_link3"/>
+    <xacro:Link reference="${prefix}right_link4"/>
+    <xacro:Link reference="${prefix}right_link5"/>
+    <xacro:Link reference="${prefix}right_link6"/>
+    <xacro:Link reference="${prefix}left_link1"/>
+    <xacro:Link reference="${prefix}left_link2"/>
+    <xacro:Link reference="${prefix}left_link3"/>
+    <xacro:Link reference="${prefix}left_link4"/>
+    <xacro:Link reference="${prefix}left_link5"/>
+    <xacro:Link reference="${prefix}left_link6"/>
+    <xacro:Link reference="${prefix}neck_link1"/>
+    <xacro:Link reference="${prefix}neck_link2"/>
+    <xacro:SimpleTransmission trans="${prefix}trans1" joint="${prefix}right_joint1" actuator="${prefix}actuator1" />
+    <xacro:SimpleTransmission trans="${prefix}trans2" joint="${prefix}right_joint2" actuator="${prefix}actuator2" />
+    <xacro:SimpleTransmission trans="${prefix}trans3" joint="${prefix}right_joint2" actuator="${prefix}actuator3" />
+    <xacro:SimpleTransmission trans="${prefix}trans4" joint="${prefix}right_joint2" actuator="${prefix}actuator4" />
+    <xacro:SimpleTransmission trans="${prefix}trans5" joint="${prefix}right_joint2" actuator="${prefix}actuator5" />
+    <xacro:SimpleTransmission trans="${prefix}trans6" joint="${prefix}right_joint2" actuator="${prefix}actuator6" />
   </xacro:macro>
 </robot>

File: avatar_description/ros2_control/follower.ros2_control.xacro (robot description, xacro)
@@ -21,6 +21,6 @@
             <param name="error_timeout_ms">500</param>
             <param name="dynamixel_model_folder">/param/dxl_model</param>
-            <param name="number_of_joints">2</param>
-            <param name="number_of_transmissions">2</param>
+            <param name="number_of_joints">14</param>
+            <param name="number_of_transmissions">14</param>
             <!-- 필수: transmission <-> joint 변환 매트릭스 (2축, 1:1 항등) -->
             <param name="transmission_to_joint_matrix">
@@ -41,6 +41,6 @@
         </hardware>
       </xacro:unless>
-      <!-- joint 2개만: joint에 ID 매핑을 넣어줌(가장 일반적인 방식) -->
-      <joint name="${prefix}joint1">
+      <!-- 오른쪽 팔 -->
+      <joint name="${prefix}right_joint1">
         <command_interface name="position"/>
         <state_interface name="position"/>
@@ -48,9 +48,83 @@
         <param name="ID">11</param>
       </joint>
-      <joint name="${prefix}joint2">
+      <joint name="${prefix}right_joint2">
         <command_interface name="position"/>
         <state_interface name="position"/>
         <state_interface name="velocity"/>
         <param name="ID">12</param>
+      </joint>
+      <joint name="${prefix}right_joint3">
+        <command_interface name="position"/>
+        <state_interface name="position"/>
+        <state_interface name="velocity"/>
+        <param name="ID">13</param>
+      </joint>
+      <joint name="${prefix}right_joint4">
+        <command_interface name="position"/>
+        <state_interface name="position"/>
+        <state_interface name="velocity"/>
+        <param name="ID">14</param>
+      </joint>
+      <joint name="${prefix}right_joint5">
+        <command_interface name="position"/>
+        <state_interface name="position"/>
+        <state_interface name="velocity"/>
+        <param name="ID">15</param>
+      </joint>
+      <joint name="${prefix}right_joint6">
+        <command_interface name="position"/>
+        <state_interface name="position"/>
+        <state_interface name="velocity"/>
+        <param name="ID">16</param>
+      </joint>
+      <!-- 왼쪽 팔 -->
+      <joint name="${prefix}left_joint1">
+        <command_interface name="position"/>
+        <state_interface name="position"/>
+        <state_interface name="velocity"/>
+        <param name="ID">21</param>
+      </joint>
+      <joint name="${prefix}left_joint2">
+        <command_interface name="position"/>
+        <state_interface name="position"/>
+        <state_interface name="velocity"/>
+        <param name="ID">22</param>
+      </joint>
+      <joint name="${prefix}left_joint3">
+        <command_interface name="position"/>
+        <state_interface name="position"/>
+        <state_interface name="velocity"/>
+        <param name="ID">23</param>
+      </joint>
+      <joint name="${prefix}left_joint4">
+        <command_interface name="position"/>
+        <state_interface name="position"/>
+        <state_interface name="velocity"/>
+        <param name="ID">24</param>
+      </joint>
+      <joint name="${prefix}left_joint5">
+        <command_interface name="position"/>
+        <state_interface name="position"/>
+        <state_interface name="velocity"/>
+        <param name="ID">25</param>
+      </joint>
+      <joint name="${prefix}left_joint6">
+        <command_interface name="position"/>
+        <state_interface name="position"/>
+        <state_interface name="velocity"/>
+        <param name="ID">26</param>
+      </joint>
+      <!-- neck joint -->
+      <joint name="${prefix}neck_joint1">
+        <command_interface name="position"/>
+        <state_interface name="position"/>
+        <state_interface name="velocity"/>
+        <param name="ID">31</param>
+      </joint>
+      <joint name="${prefix}neck_joint2">
+        <command_interface name="position"/>
+        <state_interface name="position"/>
+        <state_interface name="velocity"/>
+        <param name="ID">32</param>
       </joint>
       <!-- gpio: ID 11, 12 유지 -->
@@ -75,4 +149,232 @@
         <param name="type">dxl</param>
         <param name="ID">12</param>
+        <command_interface name="Goal Position"/>
+        <state_interface name="Present Position"/>
+        <state_interface name="Present Velocity"/>
+        <param name="Drive Mode">4</param>
+        <param name="Operating Mode">4</param>
+        <param name="Return Delay Time">0</param>
+        <param name="Min Position Limit">1024</param>
+        <param name="Max Position Limit">3140</param>
+        <param name="Min Position Limit">830</param>
+        <param name="Max Position Limit">3129</param>
+        <param name="Position P Gain">1000</param>
+        <param name="Position I Gain">0</param>
+        <param name="Position D Gain">1000</param>
+        <param name="Profile Velocity">50</param>
+        <param name="Profile Acceleration">25</param>
+      </gpio>
+      <gpio name="dxl13">
+        <param name="type">dxl</param>
+        <param name="ID">13</param>
+        <command_interface name="Goal Position"/>
+        <state_interface name="Present Position"/>
+        <state_interface name="Present Velocity"/>
+        <param name="Drive Mode">4</param>
+        <param name="Operating Mode">4</param>
+        <param name="Return Delay Time">0</param>
+        <param name="Min Position Limit">1024</param>
+        <param name="Max Position Limit">3140</param>
+        <param name="Min Position Limit">830</param>
+        <param name="Max Position Limit">3129</param>
+        <param name="Position P Gain">1000</param>
+        <param name="Position I Gain">0</param>
+        <param name="Position D Gain">1000</param>
+        <param name="Profile Velocity">50</param>
+        <param name="Profile Acceleration">25</param>
+      </gpio>
+      <gpio name="dxl14">
+        <param name="type">dxl</param>
+        <param name="ID">14</param>
+        <command_interface name="Goal Position"/>
+        <state_interface name="Present Position"/>
+        <state_interface name="Present Velocity"/>
+        <param name="Drive Mode">4</param>
+        <param name="Operating Mode">4</param>
+        <param name="Return Delay Time">0</param>
+        <param name="Min Position Limit">1024</param>
+        <param name="Max Position Limit">3140</param>
+        <param name="Min Position Limit">830</param>
+        <param name="Max Position Limit">3129</param>
+        <param name="Position P Gain">1000</param>
+        <param name="Position I Gain">0</param>
+        <param name="Position D Gain">1000</param>
+        <param name="Profile Velocity">50</param>
+        <param name="Profile Acceleration">25</param>
+      </gpio>
+      <gpio name="dxl15">
+        <param name="type">dxl</param>
+        <param name="ID">15</param>
+        <command_interface name="Goal Position"/>
+        <state_interface name="Present Position"/>
+        <state_interface name="Present Velocity"/>
+        <param name="Drive Mode">4</param>
+        <param name="Operating Mode">4</param>
+        <param name="Return Delay Time">0</param>
+        <param name="Min Position Limit">1024</param>
+        <param name="Max Position Limit">3140</param>
+        <param name="Min Position Limit">830</param>
+        <param name="Max Position Limit">3129</param>
+        <param name="Position P Gain">1000</param>
+        <param name="Position I Gain">0</param>
+        <param name="Position D Gain">1000</param>
+        <param name="Profile Velocity">50</param>
+        <param name="Profile Acceleration">25</param>
+      </gpio>
+      <gpio name="dxl16">
+        <param name="type">dxl</param>
+        <param name="ID">16</param>
+        <command_interface name="Goal Position"/>
+        <state_interface name="Present Position"/>
+        <state_interface name="Present Velocity"/>
+        <param name="Drive Mode">4</param>
+        <param name="Operating Mode">4</param>
+        <param name="Return Delay Time">0</param>
+        <param name="Min Position Limit">1024</param>
+        <param name="Max Position Limit">3140</param>
+        <param name="Min Position Limit">830</param>
+        <param name="Max Position Limit">3129</param>
+        <param name="Position P Gain">1000</param>
+        <param name="Position I Gain">0</param>
+        <param name="Position D Gain">1000</param>
+        <param name="Profile Velocity">50</param>
+        <param name="Profile Acceleration">25</param>
+      </gpio>
+      <gpio name="dxl21">
+        <param name="type">dxl</param>
+        <param name="ID">21</param>
+        <command_interface name="Goal Position"/>
+        <state_interface name="Present Position"/>
+        <state_interface name="Present Velocity"/>
+        <param name="Drive Mode">4</param>
+        <param name="Operating Mode">4</param>
+        <param name="Return Delay Time">0</param>
+        <param name="Min Position Limit">1024</param>
+        <param name="Max Position Limit">3140</param>
+        <param name="Min Position Limit">830</param>
+        <param name="Max Position Limit">3129</param>
+        <param name="Position P Gain">1000</param>
+        <param name="Position I Gain">0</param>
+        <param name="Position D Gain">1000</param>
+        <param name="Profile Velocity">50</param>
+        <param name="Profile Acceleration">25</param>
+      </gpio>
+      <gpio name="dxl22">
+        <param name="type">dxl</param>
+        <param name="ID">22</param>
+        <command_interface name="Goal Position"/>
+        <state_interface name="Present Position"/>
+        <state_interface name="Present Velocity"/>
+        <param name="Drive Mode">4</param>
+        <param name="Operating Mode">4</param>
+        <param name="Return Delay Time">0</param>
+        <param name="Min Position Limit">1024</param>
+        <param name="Max Position Limit">3140</param>
+        <param name="Min Position Limit">830</param>
+        <param name="Max Position Limit">3129</param>
+        <param name="Position P Gain">1000</param>
+        <param name="Position I Gain">0</param>
+        <param name="Position D Gain">1000</param>
+        <param name="Profile Velocity">50</param>
+        <param name="Profile Acceleration">25</param>
+      </gpio>
+      <gpio name="dxl23">
+        <param name="type">dxl</param>
+        <param name="ID">23</param>
+        <command_interface name="Goal Position"/>
+        <state_interface name="Present Position"/>
+        <state_interface name="Present Velocity"/>
+        <param name="Drive Mode">4</param>
+        <param name="Operating Mode">4</param>
+        <param name="Return Delay Time">0</param>
+        <param name="Min Position Limit">1024</param>
+        <param name="Max Position Limit">3140</param>
+        <param name="Min Position Limit">830</param>
+        <param name="Max Position Limit">3129</param>
+        <param name="Position P Gain">1000</param>
+        <param name="Position I Gain">0</param>
+        <param name="Position D Gain">1000</param>
+        <param name="Profile Velocity">50</param>
+        <param name="Profile Acceleration">25</param>
+      </gpio>
+      <gpio name="dxl24">
+        <param name="type">dxl</param>
+        <param name="ID">24</param>
+        <command_interface name="Goal Position"/>
+        <state_interface name="Present Position"/>
+        <state_interface name="Present Velocity"/>
+        <param name="Drive Mode">4</param>
+        <param name="Operating Mode">4</param>
+        <param name="Return Delay Time">0</param>
+        <param name="Min Position Limit">1024</param>
+        <param name="Max Position Limit">3140</param>
+        <param name="Min Position Limit">830</param>
+        <param name="Max Position Limit">3129</param>
+        <param name="Position P Gain">1000</param>
+        <param name="Position I Gain">0</param>
+        <param name="Position D Gain">1000</param>
+        <param name="Profile Velocity">50</param>
+        <param name="Profile Acceleration">25</param>
+      </gpio>
+      <gpio name="dxl25">
+        <param name="type">dxl</param>
+        <param name="ID">25</param>
+        <command_interface name="Goal Position"/>
+        <state_interface name="Present Position"/>
+        <state_interface name="Present Velocity"/>
+        <param name="Drive Mode">4</param>
+        <param name="Operating Mode">4</param>
+        <param name="Return Delay Time">0</param>
+        <param name="Min Position Limit">1024</param>
+        <param name="Max Position Limit">3140</param>
+        <param name="Min Position Limit">830</param>
+        <param name="Max Position Limit">3129</param>
+        <param name="Position P Gain">1000</param>
+        <param name="Position I Gain">0</param>
+        <param name="Position D Gain">1000</param>
+        <param name="Profile Velocity">50</param>
+        <param name="Profile Acceleration">25</param>
+      </gpio>
+      <gpio name="dxl26">
+        <param name="type">dxl</param>
+        <param name="ID">26</param>
+        <command_interface name="Goal Position"/>
+        <state_interface name="Present Position"/>
+        <state_interface name="Present Velocity"/>
+        <param name="Drive Mode">4</param>
+        <param name="Operating Mode">4</param>
+        <param name="Return Delay Time">0</param>
+        <param name="Min Position Limit">1024</param>
+        <param name="Max Position Limit">3140</param>
+        <param name="Min Position Limit">830</param>
+        <param name="Max Position Limit">3129</param>
+        <param name="Position P Gain">1000</param>
+        <param name="Position I Gain">0</param>
+        <param name="Position D Gain">1000</param>
+        <param name="Profile Velocity">50</param>
+        <param name="Profile Acceleration">25</param>
+      </gpio>
+      <gpio name="dxl31">
+        <param name="type">dxl</param>
+        <param name="ID">31</param>
+        <command_interface name="Goal Position"/>
+        <state_interface name="Present Position"/>
+        <state_interface name="Present Velocity"/>
+        <param name="Drive Mode">4</param>
+        <param name="Operating Mode">4</param>
+        <param name="Return Delay Time">0</param>
+        <param name="Min Position Limit">1024</param>
+        <param name="Max Position Limit">3140</param>
+        <param name="Min Position Limit">830</param>
+        <param name="Max Position Limit">3129</param>
+        <param name="Position P Gain">1000</param>
+        <param name="Position I Gain">0</param>
+        <param name="Position D Gain">1000</param>
+        <param name="Profile Velocity">50</param>
+        <param name="Profile Acceleration">25</param>
+      </gpio>
+      <gpio name="dxl32">
+        <param name="type">dxl</param>
+        <param name="ID">32</param>
         <command_interface name="Goal Position"/>
         <state_interface name="Present Position"/>

File: avatar_description/urdf/follower/follower.urdf.xacro (robot description, xacro)
@@ -19,5 +19,5 @@
   <!-- 2-DOF에는 end_effector 고정조인트가 필요 없으면 제거 가능.
        샘플 구조를 유지하기 위해 남겨두되, link2에 고정한다고 가정 -->
-  <joint name="$(arg prefix)end_effector_joint" type="fixed">
+  <!-- <joint name="$(arg prefix)end_effector_joint" type="fixed">
     <parent link="$(arg prefix)link2"/>
     <child link="$(arg prefix)end_effector_link"/>
@@ -34,5 +34,5 @@
       </material>
     </visual>
-  </link>
+  </link> -->
   <xacro:follower prefix="$(arg prefix)" />
   <xacro:follower_gazebo prefix="$(arg prefix)" />

File: avatar_description/urdf/follower/follower_arm.urdf.xacro (robot description, xacro)
@@ -2,5 +2,5 @@
 <robot xmlns:xacro="http://www.ros.org/wiki/xacro">
   <xacro:macro name="follower" params="prefix">
-    <xacro:property name="pi" value="3.1415926535" />
+    <!-- <xacro:property name="pi" value="3.1415926535" /> -->
     <xacro:property name="robot_thickness" value="0.08" />
     <xacro:property name="body_height" value="0.5" />
